Commit message: 

File: urdf/nao_h25_v32.urdf (robot description, URDF)
Before this commit: robot nao, 26 links, 25 joints
Links:
- link HeadPitch_link: geometry collision mesh filename=package://nao_detector/meshes/V32/HeadPitch.mesh scale=0.001 0.001 0.001; visual mesh filename=package://nao_detector/meshes/V32/HeadPitch.mesh scale=0.001 0.001 0.001
- link HeadYaw_link: geometry collision mesh filename=package://nao_detector/meshes/V32/HeadYaw.mesh scale=0.001 0.001 0.001; visual mesh filename=package://nao_detector/meshes/V32/HeadYaw.mesh scale=0.001 0.001 0.001
- link LAnklePitch_link: geometry collision mesh filename=package://nao_detector/meshes/V32/LAnklePitch.mesh scale=0.001 0.001 0.001; visual mesh filename=package://nao_detector/meshes/V32/LAnklePitch.mesh scale=0.001 0.001 0.001
- link LAnkleRoll_link: geometry collision mesh filename=package://nao_detector/meshes/V32/LAnkleRoll.mesh scale=0.001 0.001 0.001; visual mesh filename=package://nao_detector/meshes/V32/LAnkleRoll.mesh scale=0.001 0.001 0.001
- link LElbowRoll_link: geometry collision mesh filename=package://nao_detector/meshes/V32/LElbowRoll.mesh scale=0.001 0.001 0.001; visual mesh filename=package://nao_detector/meshes/V32/LElbowRoll.mesh scale=0.001 0.001 0.001
- link LElbowYaw_link: geometry collision mesh filename=package://nao_detector/meshes/V32/LElbowYaw.mesh scale=0.001 0.001 0.001; visual mesh filename=package://nao_detector/meshes/V32/LElbowYaw.mesh scale=0.001 0.001 0.001
- link LHipPitch_link: geometry collision mesh filename=package://nao_detector/meshes/V32/LHipPitch.mesh scale=0.001 0.001 0.001; visual mesh filename=package://nao_detector/meshes/V32/LHipPitch.mesh scale=0.001 0.001 0.001
- link LHipRoll_link: geometry collision mesh filename=package://nao_detector/meshes/V32/LHipRoll.mesh scale=0.001 0.001 0.001; visual mesh filename=package://nao_detector/meshes/V32/LHipRoll.mesh scale=0.001 0.001 0.001
- link LHipYawPitch_link: geometry collision mesh filename=package://nao_detector/meshes/V32/LHipYawPitch.mesh scale=0.001 0.001 0.001; visual mesh filename=package://nao_detector/meshes/V32/LHipYawPitch.mesh scale=0.001 0.001 0.001
- link LKneePitch_link: geometry collision mesh filename=package://nao_detector/meshes/V32/LKneePitch.mesh scale=0.001 0.001 0.001; visual mesh filename=package://nao_detector/meshes/V32/LKneePitch.mesh scale=0.001 0.001 0.001
- link LShoulderPitch_link: geometry collision mesh filename=package://nao_detector/meshes/V32/LShoulderPitch.mesh scale=0.001 0.001 0.001; visual mesh filename=package://nao_detector/meshes/V32/LShoulderPitch.mesh scale=0.001 0.001 0.001
- link LShoulderRoll_link: geometry collision mesh filename=package://nao_detector/meshes/V32/LShoulderRoll.mesh scale=0.001 0.001 0.001; visual mesh filename=package://nao_detector/meshes/V32/LShoulderRoll.mesh scale=0.001 0.001 0.001
- link LWristYaw_link: geometry collision mesh filename=package://nao_detector/meshes/V32/WristYaw.mesh scale=0.001 0.001 0.001; visual mesh filename=package://nao_detector/meshes/V32/WristYaw.mesh scale=0.001 0.001 0.001
- link RAnklePitch_link: geometry collision mesh filename=package://nao_detector/meshes/V32/RAnklePitch.mesh scale=0.001 0.001 0.001; visual mesh filename=package://nao_detector/meshes/V32/RAnklePitch.mesh scale=0.001 0.001 0.001
- link RAnkleRoll_link: geometry collision mesh filename=package://nao_detector/meshes/V32/RAnkleRoll.mesh scale=0.001 0.001 0.001; visual mesh filename=package://nao_detector/meshes/V32/RAnkleRoll.mesh scale=0.001 0.001 0.001
- link RElbowRoll_link: geometry collision mesh filename=package://nao_detector/meshes/V32/RElbowRoll.mesh scale=0.001 0.001 0.001; visual mesh filename=package://nao_detector/meshes/V32/RElbowRoll.mesh scale=0.001 0.001 0.001
- link RElbowYaw_link: geometry collision mesh filename=package://nao_detector/meshes/V32/RElbowYaw.mesh scale=0.001 0.001 0.001; visual mesh filename=package://nao_detector/meshes/V32/RElbowYaw.mesh scale=0.001 0.001 0.001
- link RHipPitch_link: geometry collision mesh filename=package://nao_detector/meshes/V32/RHipPitch.mesh scale=0.001 0.001 0.001; visual mesh filename=package://nao_detector/meshes/V32/RHipPitch.mesh scale=0.001 0.001 0.001
- link RHipRoll_link: geometry collision mesh filename=package://nao_detector/meshes/V32/RHipRoll.mesh scale=0.001 0.001 0.001; visual mesh filename=package://nao_detector/meshes/V32/RHipRoll.mesh scale=0.001 0.001 0.001
- link RHipYawPitch_link: geometry collision mesh filename=package://nao_detector/meshes/V32/RHipYawPitch.mesh scale=0.001 0.001 0.001; visual mesh filename=package://nao_detector/meshes/V32/RHipYawPitch.mesh scale=0.001 0.001 0.001
- link RKneePitch_link: geometry collision mesh filename=package://nao_detector/meshes/V32/RKneePitch.mesh scale=0.001 0.001 0.001; visual mesh filename=package://nao_detector/meshes/V32/RKneePitch.mesh scale=0.001 0.001 0.001
- link RShoulderPitch_link: geometry collision mesh filename=package://nao_detector/meshes/V32/RShoulderPitch.mesh scale=0.001 0.001 0.001; visual mesh filename=package://nao_detector/meshes/V32/RShoulderPitch.mesh scale=0.001 0.001 0.001
- link RShoulderRoll_link: geometry collision mesh filename=package://nao_detector/meshes/V32/RShoulderRoll.mesh scale=0.001 0.001 0.001; visual mesh filename=package://nao_detector/meshes/V32/RShoulderRoll.mesh scale=0.001 0.001 0.001
- link RWristYaw_link: geometry collision mesh filename=package://nao_detector/meshes/V32/WristYaw.mesh scale=0.001 0.001 0.001; visual mesh filename=package://nao_detector/meshes/V32/WristYaw.mesh scale=0.001 0.001 0.001
- link torso: geometry collision mesh filename=package://nao_detector/meshes/V32/Torso.mesh scale=0.001 0.001 0.001; visual mesh filename=package://nao_detector/meshes/V32/Torso.mesh scale=0.001 0.001 0.001
